Commit message: refactor

File: linorobot2/linorobot2_description/urdf/2wd_properties.urdf.xacro (robot description, xacro)
@@ -18,5 +18,5 @@
   </xacro:property>
   <!-- !! 3) ADDED -->
-  <xacro:property name="laser_360_pose">
+  <xacro:property name="laser_3d_pose">
     <origin xyz="0.12 0 0.50" rpy="0 0 0"/>
   </xacro:property>

File: linorobot2/linorobot2_description/urdf/robots/2wd.urdf.xacro (robot description, xacro)
@@ -55,7 +55,7 @@
   <xacro:imu/>
   <!-- !! 2) ADDED -->
-  <xacro:generic_laser_360>
-    <xacro:insert_block name="laser_360_pose" />
-  </xacro:generic_laser_360>
+  <xacro:generic_laser_3d>
+    <xacro:insert_block name="laser_3d_pose" />
+  </xacro:generic_laser_3d>
   <xacro:generic_laser>
     <xacro:insert_block name="laser_pose" />

File: linorobot2/linorobot2_description/urdf/sensors/generic_laser.urdf.xacro (robot description, xacro)
@@ -2,5 +2,6 @@
 <robot xmlns:xacro="http://ros.org/wiki/xacro">
   <xacro:include filename="$(find linorobot2_description)/urdf/sensors/laser.urdf.xacro" />
-    <xacro:include filename="$(find linorobot2_description)/urdf/sensors/laser_360.urdf.xacro" />
+  <!-- !! 1) ADDED -->
+  <xacro:include filename="$(find linorobot2_description)/urdf/sensors/laser_3d.urdf.xacro" />
   <xacro:macro name="generic_laser" params="*origin">
     <xacro:laser
@@ -32,6 +33,6 @@
   </xacro:macro>
   <!-- !! 1) ADDED -->
-  <xacro:macro name="generic_laser_360" params="*origin">
-    <xacro:laser_360
+  <xacro:macro name="generic_laser_3d" params="*origin">
+    <xacro:laser_3d
       update_rate="10"
       ray_count="360"
@@ -44,5 +45,5 @@
     >
       <xacro:insert_block name="origin" />
-    </xacro:laser_360>
+    </xacro:laser_3d>
   </xacro:macro>
 </robot>

File: linorobot2/linorobot2_description/urdf/sensors/laser_3d.urdf.xacro (robot description, xacro)
@@ -1,5 +1,5 @@
 <robot xmlns:xacro="http://ros.org/wiki/xacro">
   <xacro:property name="M_PI" value="3.1415926535897931" />
-  <xacro:macro name="laser_360" params="*origin update_rate ray_count min_angle max_angle min_range max_range frame_id topic_name">
+  <xacro:macro name="laser_3d" params="*origin update_rate ray_count min_angle max_angle min_range max_range frame_id topic_name">
     <link name="${frame_id}">
       <visual>

Commit message: 2nd depth-camera added (backside)

File: linorobot2/linorobot2_description/urdf/2wd_properties.urdf.xacro (robot description, xacro)
@@ -21,6 +21,9 @@
     <origin xyz="0.12 0 0.50" rpy="0 0 0"/>
   </xacro:property>
-  <xacro:property name="depth_sensor_pose">
+  <xacro:property name="depth_sensor_pose1">
     <origin xyz="0.14 0.0 0.045" rpy="0 0 0"/>
   </xacro:property>
+  <xacro:property name="depth_sensor_pose2">
+    <origin xyz="-0.14 0.0 0.058" rpy="0 0 3.14"/>
+  </xacro:property>
 </robot>

File: linorobot2/linorobot2_description/urdf/robots/2wd.urdf.xacro (robot description, xacro)
@@ -66,6 +66,25 @@
     <xacro:insert_block name="laser_pose" />
   </xacro:generic_laser>
-  <xacro:depth_sensor>
-    <xacro:insert_block name="depth_sensor_pose" />
+  <xacro:depth_sensor
+  	camera_link="camera_link1"
+  	camera_to_base_link="camera_to_base_link1"
+  	camera_depth_link="camera_depth_link1"
+  	camera_depth_joint="camera_depth_joint1"
+  	camera_name="camera_name1"
+  	custom_namespace="custom_namespace1"
+  	camera_controller="camera_controller1"
+  >
+    <xacro:insert_block name="depth_sensor_pose1"/>
+  </xacro:depth_sensor>
+  <xacro:depth_sensor
+  	camera_link="camera_link2"
+  	camera_to_base_link="camera_to_base_link2"
+  	camera_depth_link="camera_depth_link2"
+  	camera_depth_joint="camera_depth_joint2"
+  	camera_name="camera_name2"
+  	custom_namespace="custom_namespace2"
+  	camera_controller="camera_controller2"
+  >
+    <xacro:insert_block name="depth_sensor_pose2"/>
   </xacro:depth_sensor>
   <xacro:diff_drive_controller

File: linorobot2/linorobot2_description/urdf/sensors/depth_sensor.urdf.xacro (robot description, xacro)
@@ -1,6 +1,6 @@
 <robot xmlns:xacro="http://ros.org/wiki/xacro">
   <xacro:property name="M_PI" value="3.1415926535897931" />
-  <xacro:macro name="depth_sensor" params="*origin">
-    <link name="camera_link">
+  <xacro:macro name="depth_sensor" params="*origin camera_link camera_to_base_link camera_depth_link camera_depth_joint camera_name custom_namespace camera_controller">
+    <link name="${camera_link}">
       <visual>
         <origin xyz="0 0 0" rpy="0 0 0"/>
@@ -27,5 +27,5 @@
       </inertial>
     </link>
-    <gazebo reference="camera_link">
+    <gazebo reference="${camera_link}">
       <visual>
         <material>
@@ -37,21 +37,21 @@
       </visual>
     </gazebo>rgb(213,28,40)
-    <joint name="camera_to_base_link" type="fixed">
+    <joint name="${camera_to_base_link}" type="fixed">
       <parent link="base_link"/>
-      <child link="camera_link"/>
+      <child link="${camera_link}"/>
       <xacro:insert_block name="origin" />
     </joint>
-    <link name="camera_depth_link"/>
-    <joint name="camera_depth_joint" type="fixed">
+    <link name="${camera_depth_link}"/>
+    <joint name="${camera_depth_joint}" type="fixed">
       <origin xyz="0 0 0" rpy="-1.57 0 -1.57"/>
-      <parent link="camera_link"/>
-      <child link="camera_depth_link"/>
+      <parent link="${camera_link}"/>
+      <child link="${camera_depth_link}"/>
     </joint>
     <!-- https://github.com/ros-simulation/gazebo_ros_pkgs/wiki/ROS-2-Migration:-Camera#gazebo_ros_camera -->
-    <gazebo reference="camera_link">
-      <sensor name="camera" type="depth">
+    <gazebo reference="${camera_link}">
+      <sensor name="${camera_name}" type="depth">
         <always_on>true</always_on>
         <update_rate>1.0</update_rate>
-        <camera name="camera">
+        <camera name="${camera_name}">
           <horizontal_fov>1.50098</horizontal_fov>
           <distortion>
@@ -64,11 +64,11 @@
           </distortion>
         </camera>
-        <plugin name="camera_controller" filename="libgazebo_ros_camera.so">
+        <plugin name="${camera_controller}" filename="libgazebo_ros_camera.so">
           <ros>
-              <namespace>custom_ns</namespace>
-              <argument>camera/camera_info:=camera/color/camera_info</argument>
-              <argument>camera/image_raw:=camera/color/image_raw</argument>
-              <argument>camera/points:=camera/depth/color/points</argument>
-              <argument>camera/depth/image_raw:=camera/depth/image_rect_raw</argument>
+              <namespace>${custom_namespace}</namespace>
+              <argument>${camera_name}/camera_info:=camera/color/camera_info</argument>
+              <argument>${camera_name}/image_raw:=camera/color/image_raw</argument>
+              <argument>${camera_name}/points:=camera/depth/color/points</argument>
+              <argument>${camera_name}/depth/image_raw:=camera/depth/image_rect_raw</argument>
             <qos>
               <topic name="/camera/depth/color/points">
@@ -88,6 +88,6 @@
           <update_rate>1.0</update_rate>
           <hack_baseline>0.07</hack_baseline>
-          <frame_name>camera_depth_link</frame_name>
-          <camera_name>camera</camera_name>
+          <frame_name>${camera_depth_link}</frame_name>
+          <camera_name>${camera_name}</camera_name>
           <min_depth>0.015</min_depth>
           <max_depth>3.0</max_depth>
